Commit message: edited the file

File: rbcar_common/rbcar_description/robots/rbcar.urdf.xacro (robot description, xacro)
@@ -51,5 +51,5 @@
   	<xacro:include filename="$(find velodyne_description)/urdf/VLP-16.urdf.xacro"/>
   	<VLP-16 parent="base_link" name="velodyne" topic="/velodyne_points">
-    		<origin xyz="1.58 0 1.58" rpy="0 0 0" />
+    		<origin xyz="1.58 0 .58" rpy="0 0 0" />
   	</VLP-16>
 	<xacro:sensor_gps prefix="gps" parent="base_link">

Commit message: New changes

File: rbcar_common/rbcar_description/robots/rbcar.urdf.xacro (robot description, xacro)
@@ -6,5 +6,5 @@
 	<!-- First we import all posible elements defined in the urdf.xacro files. All these elements are defined as macro:xacros -->
 	<!-- Import Robotnik CAR base elements -->
-	<xacro:include filename="$(find rbcar_description)/urdf/bases/rbcar_base_v2.urdf.xacro" />
+	<xacro:include filename="$(find rbcar_description)/urdf/bases/rbcar_base.urdf.xacro" />
 	<!-- Import Robotnik CAR wheels -->
 	<xacro:include filename="$(find rbcar_description)/urdf/wheels/suspension_wheel_v2.urdf.xacro" />

File: rbcar_common/rbcar_description/urdf/bases/to-be-deleted/rbcar_base.urdf.xacro (robot description, xacro)
@@ -42,13 +42,13 @@
        <xacro:if value="${hq}">
        <geometry>
-	     <mesh filename="package://rbcar_description/meshes/bases/rbcar_chassis_v2.STL"/>
+	     <mesh filename="package://rbcar_description/meshes/bases/rbcar_chassis.dae"/>
        </geometry>
        </xacro:if>
        <xacro:unless value="${hq}">
        <geometry>
-	     <mesh filename="package://rbcar_description/meshes/bases/rbcar_chassis_v2.STL"/>
+	     <mesh filename="package://rbcar_description/meshes/bases/rbcar_chassis.dae"/>
        </geometry>
        </xacro:unless>
-       <material name="white">
+       <material name="darkgrey">
          <color rgba="0.1 0.1 0.1 1"/>
        </material>
@@ -57,5 +57,5 @@
        <origin xyz="0 0 0" rpy="0 0 0 " />
        <geometry>
-         <mesh filename="package://rbcar_description/meshes/bases/rbcar_chassis_v2.STL"/>
+         <mesh filename="package://rbcar_description/meshes/bases/rbcar_chassis.dae"/>
        </geometry>
     </collision>

File: rbcar_common/rbcar_description/urdf/wheels/suspension_wheel.urdf.xacro (robot description, xacro)
@@ -7,6 +7,6 @@
        axle_length. -->
   <xacro:property name="hub_dia" value="0.235"/>
-  <xacro:property name="tire_dia" value="0.470"/>
-  <xacro:property name="tire_width" value="0.2"/>
+  <xacro:property name="tire_dia" value="0.440"/>
+  <xacro:property name="tire_width" value="0.195"/>
   <xacro:property name="hex_hub_depth" value="0.120"/> <!-- or +0.072 -->
   <xacro:property name="wheel_mass" value="8.0"/>   <!-- check -->
@@ -15,6 +15,6 @@
        from a U joint to the corresponding hex hub. wheel_travel is the
        vertical wheel travel. -->
-  <xacro:property name="wheelbase" value="1.650"/>
-  <xacro:property name="hex_hub_dist" value="0.900"/>  <!-- 1.127 0.742 0.900 check -->
+  <xacro:property name="wheelbase" value="2.5"/>
+  <xacro:property name="hex_hub_dist" value="0.9191"/>  <!-- 1.127 0.742 0.900 check -->
   <xacro:property name="axle_length" value="0.120"/>
   <xacro:property name="wheel_travel" value="0.1"/>

File: rbcar_common/rbcar_description/urdf/wheels/to-be-deleted/suspension_wheel.urdf.xacro (robot description, xacro)
@@ -7,6 +7,6 @@
        axle_length. -->
   <xacro:property name="hub_dia" value="0.235"/>
-  <xacro:property name="tire_dia" value="0.440"/>
-  <xacro:property name="tire_width" value="0.195"/>
+  <xacro:property name="tire_dia" value="0.470"/>
+  <xacro:property name="tire_width" value="0.2"/>
   <xacro:property name="hex_hub_depth" value="0.120"/> <!-- or +0.072 -->
   <xacro:property name="wheel_mass" value="8.0"/>   <!-- check -->
@@ -15,6 +15,6 @@
        from a U joint to the corresponding hex hub. wheel_travel is the
        vertical wheel travel. -->
-  <xacro:property name="wheelbase" value="2.5"/>
-  <xacro:property name="hex_hub_dist" value="0.9191"/>  <!-- 1.127 0.742 0.900 check -->
+  <xacro:property name="wheelbase" value="1.650"/>
+  <xacro:property name="hex_hub_dist" value="0.900"/>  <!-- 1.127 0.742 0.900 check -->
   <xacro:property name="axle_length" value="0.120"/>
   <xacro:property name="wheel_travel" value="0.1"/>

Commit message: New changes

File: rbcar_common/rbcar_description/robots/rbcar.urdf.xacro (robot description, xacro)
@@ -77,3 +77,7 @@
         	<origin xyz="1.58 0 .25" rpy="0 0 0" />
     	</xacro:hokuyo_lx30_laser_v0>
+         <xacro:hokuyo_lx30_laser_v0 name="back_scan" parent="base" ros_topic="/rear/scan"
+    		update_rate="20" min_angle="-1.57" max_angle="1.57" >
+        	<origin xyz="-2.0 0 .25" rpy="0 0 3.14159" />
+    	</xacro:hokuyo_lx30_laser_v0>
 </robot>

Commit message: New changes

File: rbcar_common/rbcar_description/robots/rbcar.urdf.xacro (robot description, xacro)
@@ -12,5 +12,4 @@
 	<xacro:include filename="$(find robotnik_sensors)/urdf/all_sensors.urdf.xacro" />
         <!-- This adds the laser macro, including the scan for gazebo and link name -->
-	<include filename="$(find pr2_description)/urdf/sensors/hokuyo_lx30_laser.urdf.xacro" />
 	<!-- ***************** -->
 	<!-- Global parameters -->
@@ -73,11 +72,3 @@
     		<child link="camera"/>
   	</joint>
-        <xacro:hokuyo_lx30_laser_v0 name="laser_scan" parent="base" ros_topic="/base_scan/scan"
-    		update_rate="20" min_angle="-1.57" max_angle="1.57" >
-        	<origin xyz="1.58 0 .25" rpy="0 0 0" />
-    	</xacro:hokuyo_lx30_laser_v0>
-         <xacro:hokuyo_lx30_laser_v0 name="back_scan" parent="base" ros_topic="/rear/scan"
-    		update_rate="20" min_angle="-1.57" max_angle="1.57" >
-        	<origin xyz="-2.0 0 .25" rpy="0 0 3.14159" />
-    	</xacro:hokuyo_lx30_laser_v0>
 </robot>
